File: output/final_edition/boardPcb.kicad_pcb (KiCad board)
At the start: 2 copper layers, 188.6 x 119.9 mm, 118 parts

Commit message: Layout reviewed; revision 2
Connections:
- LED1 pad 2: P15 -> L024
- LED1 pad 22: P15 -> L024
- LED1 pad 4: P8 -> L023
- LED1 pad 44: P8 -> L023
- LED10 pad 2: P15 -> L016
- LED10 pad 22: P15 -> L016
- LED10 pad 4: P8 -> L015
- LED10 pad 44: P8 -> L015
- LED11 pad 2: P15 -> L010
- LED11 pad 22: P15 -> L010
- LED11 pad 4: P8 -> L009
- LED11 pad 44: P8 -> L009
- LED12 pad 2: P15 -> L004
- LED12 pad 22: P15 -> L004
- LED12 pad 4: P8 -> L003
- LED12 pad 44: P8 -> L003
- LED13 pad 2: P15 -> L021
- LED13 pad 22: P15 -> L021
- LED13 pad 4: P8 -> L020
- LED13 pad 44: P8 -> L020
- LED14 pad 2: P15 -> L015
- LED14 pad 22: P15 -> L015
- LED14 pad 4: P8 -> L014
- LED14 pad 44: P8 -> L014
- LED15 pad 2: P15 -> L009
- LED15 pad 22: P15 -> L009
- LED15 pad 4: P8 -> L008
- LED15 pad 44: P8 -> L008
- LED16 pad 2: P15 -> L003
- LED16 pad 22: P15 -> L003
- LED16 pad 4: P8 -> L002
- LED16 pad 44: P8 -> L002
- LED17 pad 2: P15 -> L020
- LED17 pad 22: P15 -> L020
- LED17 pad 4: P8 -> L019
- LED17 pad 44: P8 -> L019
- LED18 pad 2: P15 -> L014
- LED18 pad 22: P15 -> L014
- LED18 pad 4: P8 -> L013
- LED18 pad 44: P8 -> L013
- LED19 pad 2: P15 -> L008
- LED19 pad 22: P15 -> L008
- LED19 pad 4: P8 -> L007
- LED19 pad 44: P8 -> L007
- LED2 pad 2: P15 -> L018
- LED2 pad 22: P15 -> L018
- LED2 pad 4: P8 -> L017
- LED2 pad 44: P8 -> L017
- LED20 pad 2: P15 -> L002
- LED20 pad 22: P15 -> L002
- LED20 pad 4: P8 -> L001
- LED20 pad 44: P8 -> L001
- LED21 pad 2: P15 -> L019
- LED21 pad 22: P15 -> L019
- LED21 pad 4: P8 -> L018
- LED21 pad 44: P8 -> L018
- LED22 pad 2: P15 -> L013
- LED22 pad 22: P15 -> L013
- LED22 pad 4: P8 -> L012
- LED22 pad 44: P8 -> L012
- LED23 pad 2: P15 -> L007
- LED23 pad 22: P15 -> L007
- LED23 pad 4: P8 -> L006
- LED23 pad 44: P8 -> L006
- LED24 pad 2: P15 -> L001
- LED24 pad 22: P15 -> L001
- LED25 pad 2: P15 -> L029
- LED25 pad 22: P15 -> L029
- LED25 pad 4: P8 -> L028
- LED25 pad 44: P8 -> L028
- LED26 pad 2: P15 -> L028
- LED26 pad 22: P15 -> L028
- LED26 pad 4: P8 -> L027
- LED26 pad 44: P8 -> L027
- LED27 pad 2: P15 -> L027
- LED27 pad 22: P15 -> L027
- LED27 pad 4: P8 -> L026
- LED27 pad 44: P8 -> L026
- LED28 pad 2: P15 -> L026
- LED28 pad 22: P15 -> L026
- LED28 pad 4: P8 -> L025
- LED28 pad 44: P8 -> L025
- LED29 pad 2: P15 -> L025
- LED29 pad 22: P15 -> L025
- LED29 pad 4: P8 -> L024
- LED29 pad 44: P8 -> L024
- LED3 pad 2: P15 -> L012
- LED3 pad 22: P15 -> L012
- LED3 pad 4: P8 -> L011
- LED3 pad 44: P8 -> L011
- LED30 pad 2: P15 -> L024
- LED30 pad 22: P15 -> L024
- LED30 pad 4: P8 -> L023
- LED30 pad 44: P8 -> L023
- LED31 pad 2: P15 -> L018
- LED31 pad 22: P15 -> L018
- LED31 pad 4: P8 -> L017
- LED31 pad 44: P8 -> L017
- LED32 pad 2: P15 -> L012
- LED32 pad 22: P15 -> L012
- LED32 pad 4: P8 -> L011
- LED32 pad 44: P8 -> L011
- LED33 pad 2: P15 -> L006
- LED33 pad 22: P15 -> L006
- LED33 pad 4: P8 -> L005
- LED33 pad 44: P8 -> L005
- LED34 pad 2: P15 -> L023
- LED34 pad 22: P15 -> L023
- LED34 pad 4: P8 -> L022
- LED34 pad 44: P8 -> L022
- LED35 pad 2: P15 -> L017
- LED35 pad 22: P15 -> L017
- LED35 pad 4: P8 -> L016
- LED35 pad 44: P8 -> L016
- LED36 pad 2: P15 -> L011
- LED36 pad 22: P15 -> L011
- LED36 pad 4: P8 -> L010
- LED36 pad 44: P8 -> L010
- LED37 pad 2: P15 -> L005
- LED37 pad 22: P15 -> L005
- LED37 pad 4: P8 -> L004
- LED37 pad 44: P8 -> L004
- LED38 pad 2: P15 -> L022
- LED38 pad 22: P15 -> L022
- LED38 pad 4: P8 -> L021
- LED38 pad 44: P8 -> L021
- LED39 pad 2: P15 -> L016
- LED39 pad 22: P15 -> L016
- LED39 pad 4: P8 -> L015
- LED39 pad 44: P8 -> L015
- LED4 pad 2: P15 -> L006
- LED4 pad 22: P15 -> L006
- LED4 pad 4: P8 -> L005
- LED4 pad 44: P8 -> L005
- LED40 pad 2: P15 -> L010
- LED40 pad 22: P15 -> L010
- LED40 pad 4: P8 -> L009
- LED40 pad 44: P8 -> L009
- LED41 pad 2: P15 -> L004
- LED41 pad 22: P15 -> L004
- LED41 pad 4: P8 -> L003
- LED41 pad 44: P8 -> L003
- LED42 pad 2: P15 -> L021
- LED42 pad 22: P15 -> L021
- LED42 pad 4: P8 -> L020
- LED42 pad 44: P8 -> L020
- LED43 pad 2: P15 -> L015
- LED43 pad 22: P15 -> L015
- LED43 pad 4: P8 -> L014
- LED43 pad 44: P8 -> L014
- LED44 pad 2: P15 -> L009
- LED44 pad 22: P15 -> L009
- LED44 pad 4: P8 -> L008
- LED44 pad 44: P8 -> L008
- LED45 pad 2: P15 -> L003
- LED45 pad 22: P15 -> L003
- LED45 pad 4: P8 -> L002
- LED45 pad 44: P8 -> L002
- LED46 pad 2: P15 -> L020
- LED46 pad 22: P15 -> L020
- LED46 pad 4: P8 -> L019
- LED46 pad 44: P8 -> L019
- LED47 pad 2: P15 -> L014
- LED47 pad 22: P15 -> L014
- LED47 pad 4: P8 -> L013
- LED47 pad 44: P8 -> L013
- LED48 pad 2: P15 -> L008
- LED48 pad 22: P15 -> L008
- LED48 pad 4: P8 -> L007
- LED48 pad 44: P8 -> L007
- LED49 pad 2: P15 -> L002
- LED49 pad 22: P15 -> L002
- LED49 pad 4: P8 -> L001
- LED49 pad 44: P8 -> L001
- LED5 pad 2: P15 -> L023
- LED5 pad 22: P15 -> L023
- LED5 pad 4: P8 -> L022
- LED5 pad 44: P8 -> L022
- LED50 pad 2: P15 -> L019
- LED50 pad 22: P15 -> L019
- LED50 pad 4: P8 -> L018
- LED50 pad 44: P8 -> L018
- LED51 pad 2: P15 -> L013
- LED51 pad 22: P15 -> L013
- LED51 pad 4: P8 -> L012
- LED51 pad 44: P8 -> L012
- LED52 pad 2: P15 -> L007
- LED52 pad 22: P15 -> L007
- LED52 pad 4: P8 -> L006
- LED52 pad 44: P8 -> L006
- LED53 pad 2: P15 -> L001
- LED53 pad 22: P15 -> L001
- LED54 pad 2: P15 -> L029
- LED54 pad 22: P15 -> L029
- LED54 pad 4: P8 -> L028
- LED54 pad 44: P8 -> L028
- LED55 pad 2: P15 -> L028
- LED55 pad 22: P15 -> L028
- LED55 pad 4: P8 -> L027
- LED55 pad 44: P8 -> L027
- LED56 pad 2: P15 -> L027
- LED56 pad 22: P15 -> L027
- LED56 pad 4: P8 -> L026
- LED56 pad 44: P8 -> L026
- LED57 pad 2: P15 -> L026
- LED57 pad 22: P15 -> L026
- LED57 pad 4: P8 -> L025
- LED57 pad 44: P8 -> L025
- LED58 pad 2: P15 -> L025
- LED58 pad 22: P15 -> L025
- LED58 pad 4: P8 -> L024
- LED58 pad 44: P8 -> L024
- LED6 pad 2: P15 -> L017
- LED6 pad 22: P15 -> L017
- LED6 pad 4: P8 -> L016
- LED6 pad 44: P8 -> L016
- LED7 pad 2: P15 -> L011
- LED7 pad 22: P15 -> L011
- LED7 pad 4: P8 -> L010
- LED7 pad 44: P8 -> L010
- LED8 pad 2: P15 -> L005
- LED8 pad 22: P15 -> L005
- LED8 pad 4: P8 -> L004
- LED8 pad 44: P8 -> L004
- LED9 pad 2: P15 -> L022
- LED9 pad 22: P15 -> L022
- LED9 pad 4: P8 -> L021
- LED9 pad 44: P8 -> L021
Routing:
- net P15: track 879.4 -> 0.00 mm, vias 56 -> 0
- net P8: track 800.5 -> 37.0 mm, vias 37 -> 3
- net L024: track 0.00 -> 175.9 mm, vias 0 -> 4
- net L006: track 0.00 -> 144.3 mm, vias 0 -> 3
- net L012: track 0.00 -> 139.3 mm, vias 0 -> 3
- net L018: track 0.00 -> 138.7 mm, vias 0 -> 3
- net GND: track 904.8 -> 995.6 mm, vias 66 -> 35
- net L026: track 0.00 -> 62.0 mm, vias 0 -> 2
- net L002: track 0.00 -> 26.1 mm, vias 0 -> 2
- net L010: track 0.00 -> 25.9 mm, vias 0 -> 2
- net L003: track 0.00 -> 24.8 mm, vias 0 -> 2
- net L022: track 0.00 -> 24.7 mm, vias 0 -> 2
- net L008: track 0.00 -> 24.5 mm, vias 0 -> 2
- net L004: track 0.00 -> 24.4 mm, vias 0 -> 2
- net L009: track 0.00 -> 24.2 mm, vias 0 -> 2
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