File: output/pcbs/boardPcb.kicad_pcb (KiCad board)
At the start: 2 copper layers, 188.6 x 119.9 mm, 118 parts

Commit message: created custom LED footprint
Parts:
- removed LED1, LED10, LED11, LED12, LED13, LED14, LED15, LED16, LED17, LED18, LED19, LED2, LED20, LED21, LED22, LED23, LED24, LED25, LED26, LED27, LED28, LED29, LED3, LED30, LED31, LED32, LED33, LED34, LED35, LED36, LED37, LED38, LED39, LED4, LED40, LED41, LED42, LED43, LED44, LED45, LED46, LED47, LED48, LED49, LED5, LED50, LED51, LED52, LED53, LED54, LED55, LED56, LED57, LED58, LED6, LED7, LED8, LED9: , WS2812B
- added REF**: WS2812, WS2812-2020, F.Cu at (133.9, 183.2)
- added REF**: WS2812, WS2812-2020, F.Cu at (172.3, 157.2)
- added REF**: WS2812, WS2812-2020, F.Cu at (170.0, 138.4)
- added REF**: WS2812, WS2812-2020, F.Cu at (167.7, 119.5)
- added REF**: WS2812, WS2812-2020, F.Cu at (195.8, 173.5)
- added REF**: WS2812, WS2812-2020, F.Cu at (194.5, 154.6)
- added REF**: WS2812, WS2812-2020, F.Cu at (193.2, 135.6)
- added REF**: WS2812, WS2812-2020, F.Cu at (191.9, 116.7)
- added REF**: WS2812, WS2812-2020, F.Cu at (216.8, 172.1)
- added REF**: WS2812, WS2812-2020, F.Cu at (216.6, 153.1)
- added REF**: WS2812, WS2812-2020, F.Cu at (216.4, 134.1)
- added REF**: WS2812, WS2812-2020, F.Cu at (130.6, 164.5)
- added REF**: WS2812, WS2812-2020, F.Cu at (216.3, 115.1)
- added REF**: WS2812, WS2812-2020, F.Cu at (236.8, 171.9)
- added REF**: WS2812, WS2812-2020, F.Cu at (236.6, 152.9)
- added REF**: WS2812, WS2812-2020, F.Cu at (236.4, 133.9)
- added REF**: WS2812, WS2812-2020, F.Cu at (236.3, 114.9)
- added REF**: WS2812, WS2812-2020, F.Cu at (234.8, 192.5)
- added REF**: WS2812, WS2812-2020, F.Cu at (254.1, 197.5)
- added REF**: WS2812, WS2812-2020, F.Cu at (273.5, 202.5)
- added REF**: WS2812, WS2812-2020, F.Cu at (258.6, 179.6)
- added REF**: WS2812, WS2812-2020, F.Cu at (278.0, 184.6)
- added REF**: WS2812, WS2812-2020, F.Cu at (127.3, 145.8)
- added REF**: WS2812, WS2812-2020, F.Cu at (124.0, 127.1)
- added REF**: WS2812, WS2812-2020, F.Cu at (153.5, 179.8)
- added REF**: WS2812, WS2812-2020, F.Cu at (150.2, 161.1)
- added REF**: WS2812, WS2812-2020, F.Cu at (147.0, 142.3)
- added REF**: WS2812, WS2812-2020, F.Cu at (143.7, 123.6)
- added REF**: WS2812, WS2812-2020, F.Cu at (174.6, 176.1)
Connections:
- D25 pad 1: P21 -> P20
Routing:
- net (no net): track 0.00 -> 1427.5 mm
- net P4: track 39.6 -> 0.00 mm
- net P7: track 39.5 -> 0.00 mm
- net P2: track 39.5 -> 0.00 mm
- net P5: track 39.5 -> 0.00 mm
- net P6: track 39.5 -> 0.00 mm
- net P3: track 39.5 -> 0.00 mm
- net P20: track 34.6 -> 0.00 mm
- net P19: track 34.6 -> 0.00 mm
- net home2_thumb2: track 31.1 -> 0.00 mm
- net near_thumb: track 31.1 -> 0.00 mm
- net ring_number: track 31.1 -> 0.00 mm
- net pinky1_middle: track 31.1 -> 0.00 mm
- net middle_top: track 31.1 -> 0.00 mm
- net pink2_number: track 31.1 -> 0.00 mm
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Other:
- net class Default added: clearance 0.2, trace_width 0.25, via_dia 0.8, via_drill 0.4
